File: DriverCortina_Folino/DriverCortina_Folino.sch (KiCad schematic (older format))
At the start: 29 parts, among them J1 AC 220v, J2 Llave Inversora, J3 Motor 1, J4 Motor 2, K1 G3MB-202PL-DC5, K2 G3MB-202PL-DC5, Q1 BC558, Q2 BC558

Commit message: Actualización Esquemático Power_Flag
Parts:
- added FID1: Fiducial, Fiducial:Fiducial_1.5mm_Mask3mm, symbol Mechanical:Fiducial
- added H1, H2, H3, H4: MountingHole, MountingHole:MountingHole_2.5mm_Pad, symbol Mechanical:MountingHole
Other:
- moved on the sheet: C1, C3, C4, D1, D2, J1, R1, R2, R3, R4, R5
